File: PCB/viaduct/viaduct.sch (KiCad schematic (older format))
At the start: 8 parts, among them J1 n8 Bus, J2 Conn_01x03_Male, J3 Conn_01x03_Male, J4 Conn_01x10, U1 65C22S

Commit message: Close to final Viaduct and Kids' Serial cards
Changed lines of the file:
@@
 P 3300 2700
 F 0 "C1" H 3500 2675 50  0000 R CNN
-F 1 "100nf" H 3700 2775 50  0000 R CNN
+F 1 "100nf" H 3550 2775 50  0000 R CNN
 F 2 "Capacitor_THT:C_Disc_D5.0mm_W2.5mm_P2.50mm" H 3300 2700 50  0001 C CNN
 F 3 "~" H 3300 2700 50  0001 C CNN
