File: PCB/viaduct/viaduct.sch (KiCad schematic (older format))
At the start: 8 parts, among them J1 n8 Bus, J2 Conn_01x03_Male, J3 Conn_01x03_Male, J4 Conn_01x10, U1 65C22S

Commit message: Nearly final v2 PCBs
Parts:
- J2: value Conn_01x03_Male -> PORT_A_PULLUP_DOWN
- J3: value Conn_01x03_Male -> PORT_B_PULLUP_DOWN
- J4: value Conn_01x10 -> GPIO; footprint Connector_PinSocket_2.54mm:PinSocket_2x10_P2.54mm_Horizontal -> Connector_PinSocket_2.54mm:PinSocket_2x12_P2.54mm_Horizontal; symbol Connector_Generic:Conn_02x10_Odd_Even -> Connector_Generic:Conn_02x12_Odd_Even
Connections:
- net +5V: now also J4.1 (Pin_1), J4.2 (Pin_2)
- net CA1: now also J4.19 (Pin_19); no longer J4.17 (Pin_17)
- net CA2: now also J4.21 (Pin_21); no longer J4.19 (Pin_19)
- net CB1: now also J4.20 (Pin_20); no longer J4.18 (Pin_18)
- net CB2: now also J4.22 (Pin_22); no longer J4.20 (Pin_20)
- net GND: now also J4.23 (Pin_23), J4.24 (Pin_24)
- net PA0: now also J4.3 (Pin_3); no longer J4.1 (Pin_1)
- net PA1: now also J4.5 (Pin_5); no longer J4.3 (Pin_3)
- net PA2: now also J4.7 (Pin_7); no longer J4.5 (Pin_5)
- net PA3: now also J4.9 (Pin_9); no longer J4.7 (Pin_7)
- net PA4: now also J4.11 (Pin_11); no longer J4.9 (Pin_9)
- net PA5: now also J4.13 (Pin_13); no longer J4.11 (Pin_11)
- net PA6: now also J4.15 (Pin_15); no longer J4.13 (Pin_13)
- net PA7: now also J4.17 (Pin_17); no longer J4.15 (Pin_15)
- net PB0: now also J4.4 (Pin_4); no longer J4.2 (Pin_2)
- net PB1: now also J4.6 (Pin_6); no longer J4.4 (Pin_4)
- net PB2: now also J4.8 (Pin_8); no longer J4.6 (Pin_6)
- net PB3: now also J4.10 (Pin_10); no longer J4.8 (Pin_8)
- net PB4: now also J4.12 (Pin_12); no longer J4.10 (Pin_10)
- net PB5: now also J4.14 (Pin_14); no longer J4.12 (Pin_12)
- net PB6: now also J4.16 (Pin_16); no longer J4.14 (Pin_14)
- net PB7: now also J4.18 (Pin_18); no longer J4.16 (Pin_16)
- no-connect marks 9 -> 7
Changed lines of the file:
@@
 P 6825 1950
 F 0 "J2" H 6797 1882 50  0000 R CNN
-F 1 "Conn_01x03_Male" H 6797 1973 50  0000 R CNN
+F 1 "PORT_A_PULLUP_DOWN" H 6797 1973 50  0000 R CNN
 F 2 "Connector_PinHeader_2.54mm:PinHeader_1x03_P2.54mm_Vertical" H 6825 1950 50  0001 C CNN
 F 3 "~" H 6825 1950 50  0001 C CNN
@@
 P 6825 3125
 F 0 "J3" H 6797 3057 50  0000 R CNN
-F 1 "Conn_01x03_Male" H 6797 3148 50  0000 R CNN
+F 1 "PORT_B_PULLUP_DOWN" H 6797 3148 50  0000 R CNN
 F 2 "Connector_PinHeader_2.54mm:PinHeader_1x03_P2.54mm_Vertical" H 6825 3125 50  0001 C CNN
 F 3 "~" H 6825 3125 50  0001 C CNN
@@
 	2525 2300 2525 2125
 $Comp
-L Connector_Generic:Conn_02x10_Odd_Even J4
+L Connector_Generic:Conn_02x12_Odd_Even J4
 U 1 1 6064F493
-P 8275 2750
-F 0 "J4" H 8325 3367 50  0000 C CNN
-F 1 "Conn_01x10" H 8325 3276 50  0000 C CNN
-F 2 "Connector_PinSocket_2.54mm:PinSocket_2x10_P2.54mm_Horizontal" H 8275 2750 50  0001 C CNN
-F 3 "~" H 8275 2750 50  0001 C CNN
-	1    8275 2750
-	1    0    0    -1
-$EndComp
-Entry Wire Line
-	7725 2250 7825 2350
-Entry Wire Line
-	7725 2350 7825 2450
-Entry Wire Line
-	7725 2450 7825 2550
-Entry Wire Line
-	7725 2550 7825 2650
-Entry Wire Line
-	7725 2650 7825 2750
-Entry Wire Line
-	7725 2750 7825 2850
-Entry Wire Line
-	7725 2850 7825 2950
-Entry Wire Line
-	7725 2950 7825 3050
-Wire Wire Line
-	7825 2350 8075 2350
-Wire Wire Line
-	7825 2450 8075 2450
-Wire Wire Line
-	7825 2550 8075 2550
-Wire Wire Line
-	7825 2650 8075 2650
-Wire Wire Line
-	7825 2750 8075 2750
-Wire Wire Line
-	7825 2850 8075 2850
-Wire Wire Line
-	7825 2950 8075 2950
-Wire Wire Line
-	7825 3050 8075 3050
-Text Label 8000 2350 2    50   ~ 0
+P 8550 2750
+F 0 "J4" H 8600 3425 50  0000 C CNN
+F 1 "GPIO" H 8600 3350 50  0000 C CNN
+F 2 "Connector_PinSocket_2.54mm:PinSocket_2x12_P2.54mm_Horizontal" H 8550 2750 50  0001 C CNN
+F 3 "~" H 8550 2750 50  0001 C CNN
+	1    8550 2750
+	1    0    0    -1
+$EndComp
+Entry Wire Line
+	8000 2250 8100 2350
+Entry Wire Line
+	8000 2350 8100 2450
+Entry Wire Line
+	8000 2450 8100 2550
+Entry Wire Line
+	8000 2550 8100 2650
+Entry Wire Line
+	8000 2650 8100 2750
+Entry Wire Line
+	8000 2750 8100 2850
+Entry Wire Line
+	8000 2850 8100 2950
+Entry Wire Line
+	8000 2950 8100 3050
+Wire Wire Line
+	8100 2350 8350 2350
+Wire Wire Line
+	8100 2450 8350 2450
+Wire Wire Line
+	8100 2550 8350 2550
+Wire Wire Line
+	8100 2650 8350 2650
+Wire Wire Line
+	8100 2750 8350 2750
+Wire Wire Line
+	8100 2850 8350 2850
+Wire Wire Line
+	8100 2950 8350 2950
+Wire Wire Line
+	8100 3050 8350 3050
+Text Label 8275 2350 2    50   ~ 0
 PA0
-Text Label 8000 2450 2    50   ~ 0
+Text Label 8275 2450 2    50   ~ 0
 PA1
-Text Label 8000 2550 2    50   ~ 0
+Text Label 8275 2550 2    50   ~ 0
 PA2
-Text Label 8000 2650 2    50   ~ 0
+Text Label 8275 2650 2    50   ~ 0
 PA3
-Text Label 8000 2750 2    50   ~ 0
+Text Label 8275 2750 2    50   ~ 0
 PA4
-Text Label 8000 2850 2    50   ~ 0
+Text Label 8275 2850 2    50   ~ 0
 PA5
-Text Label 8000 2950 2    50   ~ 0
+Text Label 8275 2950 2    50   ~ 0
 PA6
-Text Label 8000 3050 2    50   ~ 0
+Text Label 8275 3050 2    50   ~ 0
 PA7
 Text GLabel 5025 1825 2    50   BiDi ~ 0
@@
 Wire Wire Line
 	3675 3725 3825 3725
-Text GLabel 7975 3150 0    50   BiDi ~ 0
+Text GLabel 8250 3150 0    50   BiDi ~ 0
 CA1
-Text GLabel 7975 3250 0    50   BiDi ~ 0
+Text GLabel 8250 3250 0    50   BiDi ~ 0
 CA2
 Wire Wire Line
-	7975 3150 8075 3150
-Wire Wire Line
-	7975 3250 8075 3250
-Wire Wire Line
-	8575 2350 8825 2350
-Wire Wire Line
-	8575 2450 8825 2450
-Wire Wire Line
-	8575 2550 8825 2550
-Wire Wire Line
-	8575 2650 8825 2650
-Wire Wire Line
-	8575 2750 8825 2750
-Wire Wire Line
-	8575 2850 8825 2850
-Wire Wire Line
-	8575 2950 8825 2950
-Wire Wire Line
-	8575 3050 8825 3050
-Text Label 8600 2350 0    50   ~ 0
+	8250 3150 8350 3150
+Wire Wire Line
+	8250 3250 8350 3250
+Wire Wire Line
+	8850 2350 9100 2350
+Wire Wire Line
+	8850 2450 9100 2450
+Wire Wire Line
+	8850 2550 9100 2550
+Wire Wire Line
+	8850 2650 9100 2650
+Wire Wire Line
+	8850 2750 9100 2750
+Wire Wire Line
+	8850 2850 9100 2850
+Wire Wire Line
+	8850 2950 9100 2950
+Wire Wire Line
+	8850 3050 9100 3050
+Text Label 8875 2350 0    50   ~ 0
 PB0
-Text Label 8600 2450 0    50   ~ 0
+Text Label 8875 2450 0    50   ~ 0
 PB1
-Text Label 8600 2550 0    50   ~ 0
+Text Label 8875 2550 0    50   ~ 0
 PB2
-Text Label 8600 2650 0    50   ~ 0
+Text Label 8875 2650 0    50   ~ 0
 PB3
-Text Label 8600 2750 0    50   ~ 0
+Text Label 8875 2750 0    50   ~ 0
 PB4
-Text Label 8600 2850 0    50   ~ 0
+Text Label 8875 2850 0    50   ~ 0
 PB5
-Text Label 8600 2950 0    50   ~ 0
+Text Label 8875 2950 0    50   ~ 0
 PB6
-Text Label 8600 3050 0    50   ~ 0
+Text Label 8875 3050 0    50   ~ 0
 PB7
-Text GLabel 8675 3250 2    50   BiDi ~ 0
+Text GLabel 8950 3250 2    50   BiDi ~ 0
 CB2
-Text GLabel 8675 3150 2    50   BiDi ~ 0
+Text GLabel 8950 3150 2    50   BiDi ~ 0
 CB1
 Wire Wire Line
-	8575 3150 8675 3150
-Wire Wire Line
-	8575 3250 8675 3250
-Entry Wire Line
-	8925 2350 8825 2450
-Entry Wire Line
-	8925 2250 8825 2350
-Entry Wire Line
-	8925 2450 8825 2550
-Entry Wire Line
-	8925 2550 8825 2650
-Entry Wire Line
-	8925 2650 8825 2750
-Entry Wire Line
-	8925 2750 8825 2850
-Entry Wire Line
-	8925 2850 8825 2950
-Entry Wire Line
-	8925 2950 8825 3050
+	8850 3150 8950 3150
+Wire Wire Line
+	8850 3250 8950 3250
+Entry Wire Line
+	9200 2350 9100 2450
+Entry Wire Line
+	9200 2250 9100 2350
+Entry Wire Line
+	9200 2450 9100 2550
+Entry Wire Line
+	9200 2550 9100 2650
+Entry Wire Line
+	9200 2650 9100 2750
+Entry Wire Line
+	9200 2750 9100 2850
+Entry Wire Line
+	9200 2850 9100 2950
+Entry Wire Line
+	9200 2950 9100 3050
 $Comp
 L Device:C_Small C1
@@
 Wire Wire Line
 	2675 2125 2850 2125
-NoConn ~ 2400 3600
-NoConn ~ 1900 3600
+$Comp
+L power:+5V #PWR0106
+U 1 1 605A3179
+P 8250 2250
+F 0 "#PWR0106" H 8250 2100 50  0001 C CNN
+F 1 "+5V" H 8265 2423 50  0000 C CNN
+F 2 "" H 8250 2250 50  0001 C CNN
+F 3 "" H 8250 2250 50  0001 C CNN
+	1    8250 2250
+	1    0    0    -1
+$EndComp
+Wire Wire Line
+	8350 2250 8250 2250
+Wire Wire Line
+	8350 2250 8850 2250
+Connection ~ 8350 2250
+$Comp
+L power:GND #PWR0112
+U 1 1 605B293E
+P 8250 3350
+F 0 "#PWR0112" H 8250 3100 50  0001 C CNN
+F 1 "GND" H 8255 3177 50  0000 C CNN
+F 2 "" H 8250 3350 50  0001 C CNN
+F 3 "" H 8250 3350 50  0001 C CNN
+	1    8250 3350
+	1    0    0    -1
+$EndComp
+Wire Wire Line
+	8350 3350 8250 3350
+Wire Wire Line
+	8350 3350 8850 3350
+Connection ~ 8350 3350
 Wire Bus Line
 	5125 2025 5125 2325
@@
 	5700 3025 5700 3725
 Wire Bus Line
-	7725 2250 7725 2950
-Wire Bus Line
-	8925 2250 8925 2950
+	8000 2250 8000 2950
+Wire Bus Line
+	9200 2250 9200 2950
 $EndSCHEMATC
