File: PCB/viaduct/viaduct.kicad_pcb (KiCad board)
At the start: 2 copper layers, 76.2 x 43.2 mm, 8 parts, among them J1 n8 Bus, J2 Conn_01x03_Male, J3 Conn_01x03_Male, J4 Conn_01x10, U1 65C22S

Commit message: Close to final Viaduct and Kids' Serial cards
Parts:
- moved J2 1.02 mm to (160.5, 97.0)
- moved J3 1.02 mm to (135.9, 97.0)
- moved RN1 1.02 mm to (168.1, 101.9)
- moved RN2 1.02 mm to (143.5, 101.9)
- moved U1 1.02 mm to (169.2, 108.5)
- moved C1 0.89 mm to (116.6, 108.5)
Routing:
- net +5V: track 89.8 -> 86.1 mm
- net /D7: track 21.0 -> 19.0 mm
- net CLK: track 22.8 -> 21.1 mm
- net /PA0: track 21.3 -> 20.1 mm
- net /RS1: track 53.0 -> 51.9 mm
- net R~W: track 30.5 -> 29.5 mm
- net CB2: track 62.6 -> 61.6 mm
- net /D6: track 13.3 -> 12.3 mm
- net /PB6: track 60.7 -> 59.7 mm
- net /PA4: track 27.9 -> 26.8 mm
- net /PA1: track 22.5 -> 21.5 mm
- net /PB7: track 64.3 -> 63.2 mm
- net /PA5: track 31.5 -> 30.4 mm
- net /PB5: track 57.2 -> 56.2 mm
- net /PA7: track 38.6 -> 37.6 mm
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Other:
- outline, holes or cut-outs redrawn
- board text added: "VIA"
- board text removed: "65C22S VIA"

Commit message: Nearly final v2 PCBs
Parts:
- J2: value Conn_01x03_Male -> PORT_A_PULLUP_DOWN
- J3: value Conn_01x03_Male -> PORT_B_PULLUP_DOWN
- J4: value Conn_01x10 -> GPIO; footprint Connector_PinSocket_2.54mm:PinSocket_2x10_P2.54mm_Horizontal -> Connector_PinSocket_2.54mm:PinSocket_2x12_P2.54mm_Horizontal
- moved J4 2.54 mm to (174.5, 100.1)
Connections:
- J4 pad 1: /PA0 -> +5V
- J4 pad 10: /PB4 -> /PB3
- J4 pad 11: /PA5 -> /PA4
- J4 pad 12: /PB5 -> /PB4
- J4 pad 13: /PA6 -> /PA5
- J4 pad 14: /PB6 -> /PB5
- J4 pad 15: /PA7 -> /PA6
- J4 pad 16: /PB7 -> /PB6
- J4 pad 17: CA1 -> /PA7
- J4 pad 18: CB1 -> /PB7
- J4 pad 19: CA2 -> CA1
- J4 pad 2: /PB0 -> +5V
- J4 pad 20: CB2 -> CB1
- J4 pad 3: /PA1 -> /PA0
- J4 pad 4: /PB1 -> /PB0
- J4 pad 5: /PA2 -> /PA1
- J4 pad 6: /PB2 -> /PB1
- J4 pad 7: /PA3 -> /PA2
- J4 pad 8: /PB3 -> /PB2
- J4 pad 9: /PA4 -> /PA3
Routing:
- net +5V: track 86.1 -> 111.3 mm
- net GND: vias 5 -> 4
Other:
- board text added: "+5V"
- board text added: "GND"
