File: PCB/kids serial/kids serial.sch (KiCad schematic (older format))
At the start: 6 parts, among them J1 n8 Bus Connector, J2 UARTConnector, J3 PowerViaUSB, U1 6551, X1 CXO_DIP14

Commit message: Last commit for v1
Parts:
- U1: footprint Package_DIP:DIP-28_W15.24mm -> Package_DIP:DIP-28_W15.24mm_Socket
Changed lines of the file:
@@
 F 0 "U1" H 4800 5250 50  0000 C CNN
 F 1 "6551" H 4800 5150 50  0000 C CIB
-F 2 "Package_DIP:DIP-28_W15.24mm" H 4625 3975 50  0001 C CNN
+F 2 "Package_DIP:DIP-28_W15.24mm_Socket" H 4625 3975 50  0001 C CNN
 F 3 "http://www.6502.org/documents/datasheets/mos/mos_6551_acia.pdf" H 4625 3975 50  0001 C CNN
 	1    4625 3825

Commit message: Start of Kids' Serial v2
Parts:
- removed J2: UARTConnector, Connector_PinSocket_2.54mm:PinSocket_1x06_P2.54mm_Horizontal, symbol Connector_Generic:Conn_01x06
- removed J3: PowerViaUSB, Connector_PinHeader_2.54mm:PinHeader_1x02_P2.54mm_Vertical, symbol Connector_Generic:Conn_01x02
- removed U1: 6551, Package_DIP:DIP-28_W15.24mm_Socket, symbol 65xx:6551
- added C2, C3: 100nF, Capacitor_THT:C_Disc_D5.0mm_W2.5mm_P2.50mm, symbol Device:C_Small
- added C4, C5: 47pF, Capacitor_THT:C_Disc_D3.8mm_W2.6mm_P2.50mm, symbol Device:C_Small
- added D1: TX, LED_THT:LED_D3.0mm, symbol Device:LED
- added D2: RX, LED_THT:LED_D3.0mm, symbol Device:LED
- added R1, R2: 330, Resistor_THT:R_Axial_DIN0207_L6.3mm_D2.5mm_P7.62mm_Horizontal, symbol Device:R
- added R3, R4: 27, Resistor_THT:R_Axial_DIN0207_L6.3mm_D2.5mm_P7.62mm_Horizontal, symbol Device:R
- added U1: SC28L92_PLC44, Package_LCC:PLCC-44_THT-Socket, symbol 65xx:SC28L92_PLC44
- added U2: FT230XS, Package_SO:SSOP-16_3.9x4.9mm_P0.635mm, symbol Interface_USB:FT230XS
- C1: value 100nf -> 100nF
- X1: value CXO_DIP14 -> 3.6864Mhz; footprint Oscillator:Oscillator_DIP-14 -> Oscillator:Oscillator_DIP-8; symbol Oscillator:CXO_DIP14 -> Oscillator:CXO_DIP8
Connections:
- net +5V: now also X1.8 (Vcc), C2.1, U1.44 (VCC), U2.12 (VCC); no longer X1.14 (Vcc)
- net A0: now also U1.2 (A0)
- net A1: now also U1.4 (A1)
- net A2: now also U1.6 (A2)
- net A3: now also U1.7 (A3)
- net D0: now also U1.28 (D0)
- net D1: now also U1.18 (D1)
- net D2: now also U1.27 (D2)
- net D3: now also U1.19 (D3)
- net D4: now also U1.26 (D4)
- net D5: now also U1.20 (D5)
- net D6: now also U1.25 (D6)
- net D7: now also U1.21 (D7)
- net GND: now also X1.4 (GND), C2.2, C3.2, C4.2, C5.2, U1.12 (I/M), U1.22 (GND), U2.13 (GND), U2.5 (GND); no longer X1.7 (GND)
- net R~W: now also U1.9 (~WRN)
- net XTAL_CLK: now also X1.5 (OUT), U1.36 (X1/CLK); no longer X1.8 (OUT)
- net ~CS: now also U1.39 (~CEN)
- net ~IRQ: now also U1.24 (~INTRN)
- net ~RES: now also U1.38 (RESET)
- net USB_D+: now reaches J1.26 (Pin_26)
- net USB_D+: now also C5.1, R4.2
- net USB_D-: now reaches J1.28 (Pin_28)
- net USB_D-: now also C4.1, R3.2
- new net: D2.1 (K), U2.14 (CBUS1)
- new net: D1.1 (K), U2.15 (CBUS0)
- new net: R4.1, U2.8 (USBDP)
- new net: R3.1, U2.9 (USBDM)
- new net: D1.2 (A), R1.2
- new net: D2.2 (A), R2.2
- new net +3V3: C3.1, R1.1, R2.1, U2.10 (3V3OUT), U2.11 (~RESET), U2.3 (VCCIO)
- new net RxD: U1.35 (RxDA), U2.1 (TXD)
- new net TxD: U1.33 (TxDA), U2.4 (RXD)
- new net ~CTS: U1.8 (IP0), U2.2 (~RTS)
- new net ~RTS: U1.32 (OP0), U2.6 (~CTS)
- no-connect marks 13 -> 12
Other:
- note added: "Configured for \n68xxx Bus Mode"

Commit message: Nearly final v2 PCBs
Connections:
- net CLK: no longer names the net of J1.21 (Pin_21)
- no-connect marks 12 -> 26
Changed lines of the file:
@@
 Text GLabel 950  3900 0    50   Output ~ 0
 R~W
-Text GLabel 950  4025 0    50   Output ~ 0
-CLK
 Wire Wire Line
 	1275 3800 1225 3800
@@
 Wire Wire Line
 	1275 3900 950  3900
-Wire Wire Line
-	1275 4000 1225 4000
-Wire Wire Line
-	1225 4000 1225 4025
-Wire Wire Line
-	1225 4025 950  4025
 Text GLabel 950  4150 0    50   Output ~ 0
 ~RES
@@
 Wire Wire Line
 	9700 4675 9700 4700
+NoConn ~ 4625 3100
+NoConn ~ 4625 3200
+NoConn ~ 4625 3300
+NoConn ~ 4625 3400
+NoConn ~ 4625 3500
+NoConn ~ 4625 3600
+NoConn ~ 4625 3700
+NoConn ~ 4625 4000
+NoConn ~ 4625 4100
+NoConn ~ 4625 4200
+NoConn ~ 4625 4300
+NoConn ~ 4625 4400
+NoConn ~ 4625 4500
+NoConn ~ 1275 4000
 Wire Bus Line
 	3150 2350 3150 2650
