File: PCB/n8 bit special/n8 bit special.kicad_pcb (KiCad board)
At the start: 2 copper layers, 99.7 x 97.8 mm, 36 parts, among them J1 PowerPort, J2 PORT0, J3 PORT2, J4 PORT1, J5 PORT3, J6 Conn_02x08_Odd_Even, SW1 SW_Push_Dual, U1 W65C02SxP, U2 CY62256-70PC, U3 CY62256-70PC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

Commit message: Last commit for v1
Other:
- board text added: "Reset"

Commit message: version 2 of the PCB
Parts:
- added REF1: MountingHole_3.2mm_M3_DIN965_Pad, MountingHole:MountingHole_3.2mm_M3_DIN965_Pad, F.Cu at (91.4, 128.3)
- added REF2: MountingHole_3.2mm_M3_DIN965_Pad, MountingHole:MountingHole_3.2mm_M3_DIN965_Pad, F.Cu at (137.8, 51.8)
- added REF3: MountingHole_3.2mm_M3_DIN965_Pad, MountingHole:MountingHole_3.2mm_M3_DIN965_Pad, F.Cu at (182.0, 125.9)
- C2: value 1000uF -> 470uF; footprint Capacitor_THT:CP_Radial_D10.0mm_P5.00mm -> Capacitor_THT:CP_Radial_D8.0mm_P3.80mm
- J1: value PowerPort -> USB_B_Micro; footprint Connector_PinSocket_2.54mm:PinSocket_1x04_P2.54mm_Vertical -> Connector_USB:USB_Micro-B_Amphenol_10118194_Horizontal
- X1: value 2Mhz -> 4Mhz; footprint Oscillator:Oscillator_DIP-14 -> Oscillator:Oscillator_DIP-8
- moved U1 104.1 mm to (183.8, 91.8), turned to 180 degrees
- moved U4 71.5 mm to (91.7, 43.4)
- moved C14 70.9 mm to (112.0, 43.4)
- moved C11 69.0 mm to (163.4, 89.4)
- moved R2 58.5 mm to (163.4, 76.8)
- moved U6 54.2 mm to (96.4, 88.9)
- moved C15 54.1 mm to (91.4, 83.8)
- moved R3 53.6 mm to (163.4, 72.3), turned to 90 degrees
- moved X1 28.2 mm to (180.1, 107.7), turned to 90 degrees
- moved U2 28.1 mm to (143.0, 43.4)
- moved G*** 24.3 mm to (154.7, 97.4)
- moved U3 21.8 mm to (117.3, 43.4)
- moved C1 19.2 mm to (138.2, 81.3), turned to 270 degrees
- moved U5 18.2 mm to (142.9, 88.9)
- moved R1 12.2 mm to (172.5, 137.4), turned to 90 degrees
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Connections:
- J1 pad 2: USB_D+ -> USB_D-
- J1 pad 3: USB_D- -> USB_D+
- J1 pad 4: GND -> Net-(J1-Pad4)
- X1 pad 8: CLK -> +5V
Routing:
- net /A13: track 184.3 -> 122.8 mm
- net ~IRQ: track 88.0 -> 30.3 mm
- net /D2: track 218.0 -> 169.2 mm
- net /A11: track 169.3 -> 121.2 mm, vias 0 -> 1
- net ~PORT0_CS: track 63.3 -> 17.7 mm
- net /A12: track 174.3 -> 132.7 mm, vias 0 -> 1
- net ~NMI: track 66.7 -> 26.5 mm, vias 1 -> 0
- net FUTURE0: track 99.9 -> 62.0 mm
- net /A1: track 154.4 -> 192.2 mm
- net /A9: track 166.0 -> 128.4 mm
- net ~PORT1_CS: track 67.5 -> 30.4 mm
- net /A4: track 155.6 -> 192.2 mm
- net FUTURE1: track 97.7 -> 61.8 mm
- net R~W: track 205.8 -> 170.3 mm, vias 1 -> 0
- net /A8: track 166.0 -> 135.0 mm
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Other:
- board size 99.7 x 97.8 mm -> 99.9 x 99.6 mm
- board text added: "Interrupt Handler"
- board text added: "Pullups"
- board text added: "by Nate Rivard https://github.com/nrivard/lmaos Version 2 Mar 2021"
- board text removed: "D+"
- board text removed: "D-"
- board text removed: "IRQ & NMI Handler"
- board text removed: "IRQ Pullups"
- board text removed: "JLCJLCJLCJLC"
- board text removed: "PowerPort"
- board text removed: "by Nate Rivard https://github.com/nrivard/lmaos Version 1 Mar 2021"

Commit message: Nearly final v2 PCBs
Parts:
- added C16: 100nf, Capacitor_THT:C_Disc_D5.0mm_W2.5mm_P2.50mm, F.Cu at (173.4, 113.9)
- moved G*** 2.70 mm to (156.7, 99.2)
- moved C2 2.63 mm to (175.1, 121.9), turned to 180 degrees
- moved X1 2.22 mm to (182.3, 107.6)
Routing:
- net GND: track 471.6 -> 421.5 mm
- net +5V: track 445.6 -> 448.2 mm
- net USB_D+: track 105.5 -> 104.0 mm
- net USB_D-: track 100.8 -> 99.5 mm
- net CLK: track 187.5 -> 188.1 mm
Other:
- board text added: "330"
- board text added: "3K3"

Commit message: v2 of the n8 bit special
Parts:
- moved C5 26.5 mm to (91.4, 109.5)
- moved C6 26.5 mm to (139.7, 109.5)
- moved C10 13.0 mm to (139.7, 136.1)
- moved C9 13.0 mm to (91.4, 136.1)
- moved C7 12.7 mm to (91.4, 122.8)
- moved C8 12.7 mm to (139.7, 122.8)
- moved G*** 3.62 mm to (153.4, 97.9)
- moved C4 0.95 mm to (139.7, 96.2)
- moved X1 0.91 mm to (182.1, 106.7)
- moved J2 0.89 mm to (96.5, 93.7)
- moved C2 0.60 mm to (174.8, 122.4)
- moved J4 0.57 mm to (96.5, 107.0)
- moved J3 0.25 mm to (96.5, 120.3)
- moved J1 0.19 mm to (184.0, 116.6)
- moved C1 0.13 mm to (138.3, 81.3)
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Routing:
- net ~PORT3_CS: track 97.3 -> 53.4 mm, vias 2 -> 0
- net CLK: track 188.1 -> 145.1 mm, vias 1 -> 0
- net GND: track 421.5 -> 453.3 mm, vias 11 -> 3
- net /D4: track 135.6 -> 163.7 mm
- net /A14: track 149.4 -> 128.6 mm
- net /A3: track 178.3 -> 197.7 mm, vias 1 -> 0
- net /A1: track 192.2 -> 174.2 mm
- net /D5: track 139.3 -> 155.7 mm, vias 0 -> 1
- net /A13: track 122.8 -> 107.5 mm, vias 0 -> 1
- net /A8: track 135.0 -> 120.2 mm
- net /A4: track 192.2 -> 178.6 mm, vias 2 -> 0
- net /A5: track 200.1 -> 190.0 mm, vias 0 -> 1
- net /A0: track 183.3 -> 173.7 mm
- net /A10: track 135.5 -> 126.7 mm
- net ~PORT2_CS: track 52.6 -> 61.2 mm, vias 0 -> 2
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Other:
- outline, holes or cut-outs redrawn
- net class Power: clearance 0.3 -> 0.2; trace_width 0.3 -> 0.25
- board text added: "470µF"
- board text added: "From 2 to 12 Mhz"

Commit message: v2 done
Parts:
- removed REF1, REF2, REF3: MountingHole_3.2mm_M3_DIN965_Pad, MountingHole:MountingHole_3.2mm_M3_DIN965_Pad
- moved C15 61.6 mm to (150.7, 100.4)
- moved U6 61.6 mm to (155.7, 105.5)
- moved X1 40.6 mm to (149.3, 82.9), turned to 270 degrees
- moved C1 34.3 mm to (150.7, 113.3), turned to 90 degrees
- moved C16 34.0 mm to (163.3, 81.5), turned to 270 degrees
- moved U5 32.2 mm to (155.6, 118.5)
- moved RN1 20.4 mm to (165.2, 135.9), turned to 180 degrees
- moved R2 16.5 mm to (163.3, 60.3), turned to 90 degrees
- moved G*** 15.1 mm to (143.2, 109.0)
- moved J6 13.6 mm to (162.6, 128.9), turned to 270 degrees
- moved C3 13.0 mm to (91.4, 84.1)
- moved C4 12.1 mm to (139.7, 84.1)
- moved J2 12.1 mm to (96.5, 81.6)
- moved U7 10.7 mm to (174.9, 126.0)
- moved C2 8.20 mm to (180.0, 116.1), turned to 90 degrees
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Routing:
- net FUTURE1: track 59.5 -> 114.5 mm
- net FUTURE0: track 59.3 -> 111.9 mm
- net R~W: track 169.1 -> 219.8 mm
- net ~ROM_CS: track 22.1 -> 71.9 mm
- net ~PORT0_CS: track 16.7 -> 56.4 mm
- net PORT3_NMI_PULLUP: track 85.6 -> 47.0 mm
- net PORT0_IRQ_PULLUP: track 60.8 -> 89.8 mm
- net /A10: track 126.7 -> 155.6 mm
- net /D4: track 163.7 -> 135.6 mm
- net /A14: track 128.6 -> 154.9 mm
- net ~PORT3_CS: track 53.4 -> 79.2 mm
- net ~RAM1_CS: track 64.0 -> 39.2 mm
- net /A11: track 122.4 -> 147.3 mm
- net PORT2_NMI_PULLUP: track 85.1 -> 61.4 mm
- net GND: track 453.3 -> 477.0 mm, vias 3 -> 1
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Other:
- board size 99.9 x 99.6 mm -> 99.9 x 100 mm
- net class Power: trace_width 0.25 -> 0.3

Commit message: More v2 changes
Parts:
- added G***: LOGO, graphics:MadeInAMS, F.Cu at (117.1, 125.9)
- added Q1: 2N3904, Package_TO_SOT_THT:TO-92, F.Cu at (167.8, 130.7)
- added R4: 10K, Resistor_THT:R_Axial_DIN0207_L6.3mm_D2.5mm_P7.62mm_Horizontal, F.Cu at (174.6, 128.3)
- R1: value 330 -> 220
- moved G*** 26.2 mm to (117.0, 108.6)
- moved R1 8.70 mm to (178.8, 128.3)
- moved U7 7.36 mm to (167.8, 124.4)
- moved C2 1.35 mm to (181.0, 115.2)
- moved D1 0.92 mm to (173.5, 136.2)
- moved SW1 0.32 mm to (177.8, 132.4)
Connections:
- D1 pad 2: ~RES -> Net-(D1-Pad2)
Routing:
- net GND: track 477.0 -> 457.9 mm, vias 1 -> 4
- net +5V: track 461.7 -> 470.7 mm
- net Net-(Q1-Pad2): track 0.00 -> 8.60 mm
- net Net-(D1-Pad2): track 0.00 -> 6.99 mm
- net ~RES: track 167.4 -> 172.3 mm
- net Net-(D1-Pad1): track 6.47 -> 10.1 mm
- net /A0: track 173.5 -> 170.8 mm
- net /D5: track 141.1 -> 139.0 mm
- net /D4: track 135.6 -> 134.3 mm
- net /D6: track 144.8 -> 143.8 mm
- net FUTURE0: track 111.9 -> 110.9 mm
- net USB_D+: track 116.5 -> 117.3 mm
- net /D2: track 158.7 -> 157.9 mm
- net PORT0_IRQ_PULLUP: track 89.8 -> 90.4 mm
- net /D3: track 131.8 -> 131.2 mm
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Other:
- board text added: "10K"
- board text added: "220"
- board text removed: "330"
