File: PCB/n8 bit special/n8 bit special.sch (KiCad schematic (older format))
At the start: 35 parts, among them J1 PowerPort, J2 PORT0, J3 PORT2, J4 PORT1, J5 PORT3, J6 Conn_02x08_Odd_Even, SW1 SW_Push_Dual, U1 W65C02SxP, U2 CY62256-70PC, U3 CY62256-70PC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

Commit message: version 2 of the PCB
Parts:
- removed J1: PowerPort, Connector_PinSocket_2.54mm:PinSocket_1x04_P2.54mm_Vertical, symbol Connector_Generic:Conn_01x04
- added J1: USB_B_Micro, Connector_USB:USB_Micro-B_Amphenol_10118194_Horizontal, symbol Connector:USB_B_Micro
- C2: value 1000uF -> 470uF; footprint Capacitor_THT:CP_Radial_D10.0mm_P5.00mm -> Capacitor_THT:CP_Radial_D8.0mm_P3.80mm
- X1: value 2Mhz -> 4Mhz; footprint Oscillator:Oscillator_DIP-14 -> Oscillator:Oscillator_DIP-8; symbol Oscillator:CXO_DIP14 -> Oscillator:CXO_DIP8
Connections:
- net +5V: now also X1.8 (Vcc), J1.1 (VBUS); no longer X1.14 (Vcc)
- net CLK: now also X1.5 (OUT); no longer X1.8 (OUT)
- net GND: now also X1.4 (GND), J1.5 (GND), J1.6 (Shield); no longer X1.7 (GND)
- net USB_D+: now also J1.3 (D+)
- net USB_D-: now also J1.2 (D-)
- no-connect marks 7 -> 9
Other:
- moved on the sheet: C2
Changed lines of the file:
@@
 	1725 3875 1950 3875
-$Comp
-L Oscillator:CXO_DIP14 X1
-U 1 1 6041F292
-P 1425 3875
-F 0 "X1" H 1725 3925 50  0000 L CNN
-F 1 "2Mhz" H 1725 3825 50  0000 L CNN
-F 2 "Oscillator:Oscillator_DIP-14" H 1875 3525 50  0001 C CNN
-F 3 "http://cdn-reichelt.de/documents/datenblatt/B400/OSZI.pdf" H 1325 3875 50  0001 C CNN
-	1    1425 3875
-	1    0    0    -1
-$EndComp
 $Comp
 L power:GND #PWR0114
@@
 $EndComp
 $Comp
-L Device:CP C2
-U 1 1 61A18110
-P 1150 1750
-F 0 "C2" H 925 1800 50  0000 L CNN
-F 1 "1000uF" H 750 1700 50  0000 L CNN
-F 2 "Capacitor_THT:CP_Radial_D10.0mm_P5.00mm" H 1188 1600 50  0001 C CNN
-F 3 "~" H 1150 1750 50  0001 C CNN
-	1    1150 1750
-	1    0    0    -1
-$EndComp
-Wire Wire Line
-	1150 1900 1025 1900
-Connection ~ 1150 1900
-Wire Wire Line
-	1150 1600 1025 1600
-Connection ~ 1150 1600
-$Comp
-L power:PWR_FLAG #FLG0101
-U 1 1 6177EEDC
-P 1675 1600
-F 0 "#FLG0101" H 1675 1675 50  0001 C CNN
-F 1 "PWR_FLAG" H 1675 1773 50  0000 C CNN
-F 2 "" H 1675 1600 50  0001 C CNN
-F 3 "~" H 1675 1600 50  0001 C CNN
-	1    1675 1600
-	1    0    0    -1
-$EndComp
-Wire Wire Line
-	1700 1800 1675 1800
-Wire Wire Line
-	1700 1700 1675 1700
-Text GLabel 1675 1700 0    50   BiDi ~ 0
-USB_D+
-Text GLabel 1675 1800 0    50   BiDi ~ 0
-USB_D-
-Wire Wire Line
-	1700 1900 1675 1900
-Wire Wire Line
-	1700 1600 1675 1600
-$Comp
-L power:GND #PWR0143
-U 1 1 614EE1DF
-P 1025 1900
-F 0 "#PWR0143" H 1025 1650 50  0001 C CNN
-F 1 "GND" H 1030 1727 50  0000 C CNN
-F 2 "" H 1025 1900 50  0001 C CNN
-F 3 "" H 1025 1900 50  0001 C CNN
-	1    1025 1900
-	1    0    0    -1
-$EndComp
-$Comp
-L power:+5V #PWR0142
-U 1 1 61491882
-P 1025 1600
-F 0 "#PWR0142" H 1025 1450 50  0001 C CNN
-F 1 "+5V" H 1040 1773 50  0000 C CNN
-F 2 "" H 1025 1600 50  0001 C CNN
-F 3 "" H 1025 1600 50  0001 C CNN
-	1    1025 1600
-	1    0    0    -1
-$EndComp
-$Comp
-L Connector_Generic:Conn_01x04 J1
-U 1 1 614904B3
-P 1900 1700
-F 0 "J1" H 1980 1692 50  0000 L CNN
-F 1 "PowerPort" H 1980 1601 50  0000 L CNN
-F 2 "Connector_PinSocket_2.54mm:PinSocket_1x04_P2.54mm_Vertical" H 1900 1700 50  0001 C CNN
-F 3 "~" H 1900 1700 50  0001 C CNN
-	1    1900 1700
-	1    0    0    -1
-$EndComp
-$Comp
 L power:GND #PWR0102
 U 1 1 60412457
@@
 	9500 3250 9500 3200
 Connection ~ 9500 3200
-$Comp
-L power:PWR_FLAG #FLG0102
-U 1 1 6232E9D2
-P 1675 1900
-F 0 "#FLG0102" H 1675 1975 50  0001 C CNN
-F 1 "PWR_FLAG" H 1675 2073 50  0000 C CNN
-F 2 "" H 1675 1900 50  0001 C CNN
-F 3 "~" H 1675 1900 50  0001 C CNN
-	1    1675 1900
-	-1   0    0    1
-$EndComp
-Connection ~ 1675 1900
-Wire Wire Line
-	1675 1900 1150 1900
-Connection ~ 1675 1600
-Wire Wire Line
-	1675 1600 1150 1600
 Wire Notes Line
 	2525 2500 650  2500
@@
 	0    1    1    0
 $EndComp
+Text Label 8650 2825 1    50   ~ 0
+A[0..15]
+Text GLabel 1475 1675 2    50   BiDi ~ 0
+USB_D+
+Text GLabel 1475 1775 2    50   BiDi ~ 0
+USB_D-
+$Comp
+L power:GND #PWR0143
+U 1 1 614EE1DF
+P 2150 2075
+F 0 "#PWR0143" H 2150 1825 50  0001 C CNN
+F 1 "GND" H 2155 1902 50  0000 C CNN
+F 2 "" H 2150 2075 50  0001 C CNN
+F 3 "" H 2150 2075 50  0001 C CNN
+	1    2150 2075
+	1    0    0    -1
+$EndComp
+$Comp
+L power:+5V #PWR0142
+U 1 1 61491882
+P 2150 1475
+F 0 "#PWR0142" H 2150 1325 50  0001 C CNN
+F 1 "+5V" H 2165 1648 50  0000 C CNN
+F 2 "" H 2150 1475 50  0001 C CNN
+F 3 "" H 2150 1475 50  0001 C CNN
+	1    2150 1475
+	1    0    0    -1
+$EndComp
+$Comp
+L Connector:USB_B_Micro J1
+U 1 1 605493AE
+P 1050 1675
+F 0 "J1" H 1107 2142 50  0000 C CNN
+F 1 "USB_B_Micro" H 1107 2051 50  0000 C CNN
+F 2 "Connector_USB:USB_Micro-B_Amphenol_10118194_Horizontal" H 1200 1625 50  0001 C CNN
+F 3 "~" H 1200 1625 50  0001 C CNN
+	1    1050 1675
+	1    0    0    -1
+$EndComp
+Wire Wire Line
+	1350 1675 1475 1675
+Wire Wire Line
+	1350 1775 1475 1775
+$Comp
+L Device:CP C2
+U 1 1 61A18110
+P 2050 1775
+F 0 "C2" H 2275 1850 50  0000 L CNN
+F 1 "470uF" H 2200 1750 50  0000 L CNN
+F 2 "Capacitor_THT:CP_Radial_D8.0mm_P3.80mm" H 2088 1625 50  0001 C CNN
+F 3 "~" H 2050 1775 50  0001 C CNN
+	1    2050 1775
+	1    0    0    -1
+$EndComp
+Wire Wire Line
+	2050 1625 2050 1475
+Connection ~ 2050 1475
+Wire Wire Line
+	2050 1475 2150 1475
+Wire Wire Line
+	2050 1925 2050 2075
+Connection ~ 2050 2075
+Wire Wire Line
+	2050 2075 2150 2075
+NoConn ~ 1350 1875
+$Comp
+L Oscillator:CXO_DIP8 X1
+U 1 1 6041F292
+P 1425 3875
+F 0 "X1" H 1725 3925 50  0000 L CNN
+F 1 "4Mhz" H 1725 3825 50  0000 L CNN
+F 2 "Oscillator:Oscillator_DIP-8" H 1875 3525 50  0001 C CNN
+F 3 "http://cdn-reichelt.de/documents/datenblatt/B400/OSZI.pdf" H 1325 3875 50  0001 C CNN
+	1    1425 3875
+	1    0    0    -1
+$EndComp
+NoConn ~ 1500 3775
+Wire Wire Line
+	1050 2075 2050 2075
+Wire Wire Line
+	1350 1475 2050 1475
+Wire Wire Line
+	950  2075 1050 2075
 Wire Bus Line
 	6375 8950 6375 9450
@@
 Wire Bus Line
 	13625 1425 13625 2825
-Text Label 8650 2825 1    50   ~ 0
-A[0..15]
+Connection ~ 1050 2075
 $EndSCHEMATC

Commit message: Nearly final v2 PCBs
Parts:
- added C16: 100nf, Capacitor_THT:C_Disc_D5.0mm_W2.5mm_P2.50mm, symbol Device:C_Small
Connections:
- net +5V: now also C16.2
- net GND: now also C16.1; no longer J1.6 (Shield)
- no-connect marks 9 -> 10
Other:
- moved on the sheet: X1
Changed lines of the file:
@@
 L power:GND #PWR0112
 U 1 1 60420A5A
-P 1425 4250
-F 0 "#PWR0112" H 1425 4000 50  0001 C CNN
-F 1 "GND" H 1430 4077 50  0000 C CNN
-F 2 "" H 1425 4250 50  0001 C CNN
-F 3 "" H 1425 4250 50  0001 C CNN
-	1    1425 4250
+P 1625 4300
+F 0 "#PWR0112" H 1625 4050 50  0001 C CNN
+F 1 "GND" H 1630 4127 50  0000 C CNN
+F 2 "" H 1625 4300 50  0001 C CNN
+F 3 "" H 1625 4300 50  0001 C CNN
+	1    1625 4300
 	1    0    0    -1
 $EndComp
@@
 L power:+5V #PWR0113
 U 1 1 604216C0
-P 1425 3475
-F 0 "#PWR0113" H 1425 3325 50  0001 C CNN
-F 1 "+5V" H 1440 3648 50  0000 C CNN
-F 2 "" H 1425 3475 50  0001 C CNN
-F 3 "" H 1425 3475 50  0001 C CNN
-	1    1425 3475
-	1    0    0    -1
-$EndComp
-Wire Wire Line
-	1425 3475 1425 3575
-Wire Wire Line
-	1425 4175 1425 4250
-NoConn ~ 1125 3875
-Text GLabel 1950 3875 2    50   Output ~ 0
+P 1625 3525
+F 0 "#PWR0113" H 1625 3375 50  0001 C CNN
+F 1 "+5V" H 1640 3698 50  0000 C CNN
+F 2 "" H 1625 3525 50  0001 C CNN
+F 3 "" H 1625 3525 50  0001 C CNN
+	1    1625 3525
+	1    0    0    -1
+$EndComp
+Wire Wire Line
+	1625 3525 1625 3575
+Wire Wire Line
+	1625 4225 1625 4275
+NoConn ~ 1325 3925
+Text GLabel 2150 3925 2    50   Output ~ 0
 CLK
 Wire Wire Line
-	1725 3875 1950 3875
+	1925 3925 2150 3925
 $Comp
 L power:GND #PWR0114
@@
 L Oscillator:CXO_DIP8 X1
 U 1 1 6041F292
-P 1425 3875
-F 0 "X1" H 1725 3925 50  0000 L CNN
-F 1 "4Mhz" H 1725 3825 50  0000 L CNN
-F 2 "Oscillator:Oscillator_DIP-8" H 1875 3525 50  0001 C CNN
-F 3 "http://cdn-reichelt.de/documents/datenblatt/B400/OSZI.pdf" H 1325 3875 50  0001 C CNN
-	1    1425 3875
-	1    0    0    -1
-$EndComp
-NoConn ~ 1500 3775
+P 1625 3925
+F 0 "X1" H 1925 3975 50  0000 L CNN
+F 1 "4Mhz" H 1925 3875 50  0000 L CNN
+F 2 "Oscillator:Oscillator_DIP-8" H 2075 3575 50  0001 C CNN
+F 3 "http://cdn-reichelt.de/documents/datenblatt/B400/OSZI.pdf" H 1525 3925 50  0001 C CNN
+	1    1625 3925
+	1    0    0    -1
+$EndComp
+NoConn ~ 1700 3825
 Wire Wire Line
 	1050 2075 2050 2075
 Wire Wire Line
 	1350 1475 2050 1475
-Wire Wire Line
-	950  2075 1050 2075
+$Comp
+L Device:C_Small C16
+U 1 1 6059534A
+P 1075 3900
+F 0 "C16" H 1275 3875 50  0000 R CNN
+F 1 "100nf" H 1325 3975 50  0000 R CNN
+F 2 "Capacitor_THT:C_Disc_D5.0mm_W2.5mm_P2.50mm" H 1075 3900 50  0001 C CNN
+F 3 "~" H 1075 3900 50  0001 C CNN
+	1    1075 3900
+	-1   0    0    1
+$EndComp
+Wire Wire Line
+	1625 3575 1075 3575
+Wire Wire Line
+	1075 3575 1075 3800
+Connection ~ 1625 3575
+Wire Wire Line
+	1625 3575 1625 3625
+Wire Wire Line
+	1075 4000 1075 4275
+Wire Wire Line
+	1075 4275 1625 4275
+Connection ~ 1625 4275
+Wire Wire Line
+	1625 4275 1625 4300
+NoConn ~ 950  2075
 Wire Bus Line
 	6375 8950 6375 9450
@@
 Wire Bus Line
 	13625 1425 13625 2825
-Connection ~ 1050 2075
 $EndSCHEMATC

Commit message: v2 of the n8 bit special
Parts:
- renumbered C7 to C5, C8 to C6, C5 to C7, C6 to C8
Changed lines of the file:
@@
 	7275 6125 7650 6125
 $Comp
-L Device:C_Small C8
+L Device:C_Small C6
 U 1 1 633D5C80
 P 6875 7975
-F 0 "C8" V 6646 7975 50  0000 C CNN
+F 0 "C6" V 6646 7975 50  0000 C CNN
 F 1 "100nf" V 6737 7975 50  0000 C CNN
 F 2 "Capacitor_THT:C_Disc_D5.0mm_W2.5mm_P2.50mm" H 6875 7975 50  0001 C CNN
@@
 $EndComp
 $Comp
-L Device:C_Small C7
+L Device:C_Small C5
 U 1 1 633D5C86
 P 6875 5800
-F 0 "C7" V 6646 5800 50  0000 C CNN
+F 0 "C5" V 6646 5800 50  0000 C CNN
 F 1 "100nf" V 6737 5800 50  0000 C CNN
 F 2 "Capacitor_THT:C_Disc_D5.0mm_W2.5mm_P2.50mm" H 6875 5800 50  0001 C CNN
@@
 	4375 8850 4750 8850
 $Comp
-L Device:C_Small C6
+L Device:C_Small C8
 U 1 1 6341904F
 P 3975 10700
-F 0 "C6" V 3746 10700 50  0000 C CNN
+F 0 "C8" V 3746 10700 50  0000 C CNN
 F 1 "100nf" V 3837 10700 50  0000 C CNN
 F 2 "Capacitor_THT:C_Disc_D5.0mm_W2.5mm_P2.50mm" H 3975 10700 50  0001 C CNN
@@
 $EndComp
 $Comp
-L Device:C_Small C5
+L Device:C_Small C7
 U 1 1 63419055
 P 3975 8525
-F 0 "C5" V 3746 8525 50  0000 C CNN
+F 0 "C7" V 3746 8525 50  0000 C CNN
 F 1 "100nf" V 3837 8525 50  0000 C CNN
 F 2 "Capacitor_THT:C_Disc_D5.0mm_W2.5mm_P2.50mm" H 3975 8525 50  0001 C CNN

Commit message: More v2 changes
Parts:
- added Q1: 2N3904, Package_TO_SOT_THT:TO-92, symbol Transistor_BJT:2N3904
- added R4: 10K, Resistor_THT:R_Axial_DIN0207_L6.3mm_D2.5mm_P7.62mm_Horizontal, symbol Device:R
- R1: value 330 -> 220
Connections:
- net +5V: now also Q1.3 (C)
- net ~RES: now also R4.2; no longer D1.2 (A)
- new net: D1.2 (A), Q1.1 (E)
- new net: Q1.2 (B), R4.1
Other:
- moved on the sheet: D1, R1
Changed lines of the file:
@@
 	1    0    0    -1
 $EndComp
-Text GLabel 4650 1650 2    50   Output ~ 0
+Text GLabel 4425 1650 2    50   Output ~ 0
 ~RES
 $Comp
@@
 L Device:LED_ALT D1
 U 1 1 6045033F
-P 4275 1300
-F 0 "D1" H 4268 1517 50  0000 C CNN
-F 1 "LED_ALT" H 4268 1426 50  0000 C CNN
-F 2 "LED_THT:LED_D3.0mm" H 4275 1300 50  0001 C CNN
-F 3 "~" H 4275 1300 50  0001 C CNN
-	1    4275 1300
-	-1   0    0    1
+P 5000 1750
+F 0 "D1" H 4993 1967 50  0000 C CNN
+F 1 "LED_ALT" H 4993 1876 50  0000 C CNN
+F 2 "LED_THT:LED_D3.0mm" H 5000 1750 50  0001 C CNN
+F 3 "~" H 5000 1750 50  0001 C CNN
+	1    5000 1750
+	0    -1   -1   0
 $EndComp
 $Comp
 L power:GND #PWR0128
 U 1 1 60450336
-P 4900 1300
-F 0 "#PWR0128" H 4900 1050 50  0001 C CNN
-F 1 "GND" H 4905 1127 50  0000 C CNN
-F 2 "" H 4900 1300 50  0001 C CNN
-F 3 "" H 4900 1300 50  0001 C CNN
-	1    4900 1300
+P 5000 2325
+F 0 "#PWR0128" H 5000 2075 50  0001 C CNN
+F 1 "GND" H 4850 2250 50  0000 C CNN
+F 2 "" H 5000 2325 50  0001 C CNN
+F 3 "" H 5000 2325 50  0001 C CNN
+	1    5000 2325
 	1    0    0    -1
 $EndComp
@@
 L Device:R R1
 U 1 1 60450330
-P 4650 1300
-F 0 "R1" V 4550 1300 50  0000 C CNN
-F 1 "330" V 4650 1300 50  0000 C CNN
-F 2 "Resistor_THT:R_Axial_DIN0207_L6.3mm_D2.5mm_P7.62mm_Horizontal" H 4650 1300 50  0001 C CNN
-F 3 "~" H 4650 1300 50  0001 C CNN
-	1    4650 1300
-	0    -1   -1   0
-$EndComp
-Wire Wire Line
-	4425 1300 4500 1300
-Wire Wire Line
-	4800 1300 4900 1300
+P 5000 2125
+F 0 "R1" V 4900 2125 50  0000 C CNN
+F 1 "220" V 5000 2125 50  0000 C CNN
+F 2 "Resistor_THT:R_Axial_DIN0207_L6.3mm_D2.5mm_P7.62mm_Horizontal" H 5000 2125 50  0001 C CNN
+F 3 "~" H 5000 2125 50  0001 C CNN
+	1    5000 2125
+	1    0    0    -1
+$EndComp
+Wire Wire Line
+	5000 1900 5000 1975
+Wire Wire Line
+	5000 2275 5000 2325
 Wire Notes Line
 	8550 875  8550 3900
@@
 Connection ~ 3975 1650
 Wire Wire Line
-	3975 1650 4075 1650
-Wire Wire Line
 	4500 2025 4500 2075
-Wire Wire Line
-	4075 1300 4075 1650
-Connection ~ 4075 1650
-Wire Wire Line
-	4075 1650 4650 1650
-Wire Wire Line
-	4075 1300 4125 1300
 Wire Notes Line
 	5400 875  5400 2500
@@
 	1625 4275 1625 4300
 NoConn ~ 950  2075
+Wire Wire Line
+	3975 1650 4425 1650
+$Comp
+L Transistor_BJT:2N3904 Q1
+U 1 1 60DCF972
+P 4900 1300
+F 0 "Q1" H 5090 1346 50  0000 L CNN
+F 1 "2N3904" H 5090 1255 50  0000 L CNN
+F 2 "Package_TO_SOT_THT:TO-92" H 5100 1225 50  0001 L CIN
+F 3 "https://www.onsemi.com/pub/Collateral/2N3903-D.PDF" H 4900 1300 50  0001 L CNN
+	1    4900 1300
+	1    0    0    -1
+$EndComp
+Wire Wire Line
+	4600 1300 4700 1300
+$Comp
+L power:+5V #PWR01
+U 1 1 611B59A4
+P 5000 1025
+F 0 "#PWR01" H 5000 875 50  0001 C CNN
+F 1 "+5V" H 4875 1100 50  0000 C CNN
+F 2 "" H 5000 1025 50  0001 C CNN
+F 3 "" H 5000 1025 50  0001 C CNN
+	1    5000 1025
+	1    0    0    -1
+$EndComp
+Wire Wire Line
+	5000 1025 5000 1100
+Wire Wire Line
+	5000 1500 5000 1600
+$Comp
+L Device:R R4
+U 1 1 60DD1216
+P 4450 1300
+F 0 "R4" V 4350 1300 50  0000 C CNN
+F 1 "10K" V 4450 1300 50  0000 C CNN
+F 2 "Resistor_THT:R_Axial_DIN0207_L6.3mm_D2.5mm_P7.62mm_Horizontal" H 4450 1300 50  0001 C CNN
+F 3 "~" H 4450 1300 50  0001 C CNN
+	1    4450 1300
+	0    1    1    0
+$EndComp
+Wire Wire Line
+	3975 1650 3975 1300
+Wire Wire Line
+	3975 1300 4300 1300
 Wire Bus Line
 	6375 8950 6375 9450
